File: Synchronous Buck-Boost Converter.kicad_sch (KiCad schematic)
At the start: 12 parts, among them J1 Conn_01x06_Pin, Q1 NMOS, Q2 NMOS, Q3 NMOS, Q4 NMOS, U1 IR2110, U2 STM32G4A1CETx, U3 INA240A3D

Commit message: Bidirectionnal Sychronous 4 Switch BB Hardware V1
Parts:
- removed J1: Conn_01x06_Pin, Connector_PinSocket_1.27mm:PinSocket_1x06_P1.27mm_Vertical, symbol Connector:Conn_01x06_Pin
- removed Q1, Q2, Q3, Q4: NMOS, Package_TO_SOT_THT:TO-220-3_Horizontal_TabDown, symbol Simulation_SPICE:NMOS
- removed U1: IR2110, Package_DIP:DIP-14_W7.62mm, symbol Driver_FET:IR2110
- removed U2: STM32G4A1CETx, Package_QFP:LQFP-48_7x7mm_P0.5mm, symbol MCU_ST_STM32G4:STM32G4A1CETx
- added C10, C9: 0.1u, Capacitor_SMD:C_0603_1608Metric, symbol Device:C
- added C11, C8: 1u, Capacitor_SMD:C_1206_3216Metric, symbol Device:C
- added C12, C7: 4.7u, Capacitor_SMD:C_1210_3225Metric, symbol Device:C
- added C13, C14, C15, C23, C36, C38, C4, C5, C6: 10u, Capacitor_SMD:C_1210_3225Metric, symbol Device:C
- added C16, C3: 100u, Capacitor_SMD:C_Elec_10x10.2, symbol Device:C_US
- added C17, C18, C22: 1n, Capacitor_SMD:C_0603_1608Metric, symbol Device:C
- added C19, C52, C53: 10n, Capacitor_SMD:C_0603_1608Metric, symbol Device:C
- added C2: 5.6n, Capacitor_SMD:C_1206_3216Metric, symbol Device:C
- added C20, C31, C32, C41, C42, C43, C44, C45, C50: 100n, Capacitor_SMD:C_0805_2012Metric, symbol Device:C
- added C21: 1u, Capacitor_SMD:C_0805_2012Metric, symbol Device:C
- added C27, C37: 2.2u, Capacitor_SMD:C_0805_2012Metric, symbol Device:C
- added C39, C40, C46: 4.7u, Capacitor_SMD:C_0805_2012Metric, symbol Device:C
- added C47, C49: 18p, Capacitor_SMD:C_0402_1005Metric, symbol Device:C
- added D2, D3, D4: SKL16, Diode_SMD:Nexperia_CFP3_SOD-123W, symbol Device:D
- added D5, D6: 70V, Diode_SMD:D_SMA, symbol Device:D_TVS
- added D7, D8: 60V 1A, Diode_SMD:D_MicroSMP_AK, symbol Device:D_Schottky
- added F1, F2: 15A, Fuse:Fuse_2512_6332Metric_Pad1.52x3.35mm_HandSolder, symbol Device:Fuse_Small
- added FB1: 600R, Inductor_SMD:L_0603_1608Metric, symbol Device:FerriteBead
- added H1, H2, H3, H4: MountingHole_Pad, MountingHole:MountingHole_4.3mm_M4_Pad_Via, symbol Mechanical:MountingHole_Pad
- added J1, J2: Screw_Terminal_01x02, TerminalBlock_Phoenix:TerminalBlock_Phoenix_MKDS-1,5-2-5.08_1x02_P5.08mm_Horizontal, symbol Connector:Screw_Terminal_01x02
- added J4: Conn_01x16_Pin, Connector_PinHeader_2.54mm:PinHeader_1x16_P2.54mm_Vertical, symbol Connector:Conn_01x16_Pin
- added Q1, Q2, Q3, Q4: SiR182DP, Mosfets:PowerPAK_SO-8_Single, symbol Transistor_FET:SiR696DP
- added R10, R7, R8, R9: 5.11, Resistor_SMD:R_0805_2012Metric, symbol Device:R
- added R11, R12: 3.3, Resistor_SMD:R_2512_6332Metric, symbol Device:R
- added R13, R16: 4k7R, Resistor_SMD:R_0805_2012Metric, symbol Device:R
- added R17, R18: 1kR, Resistor_SMD:R_0805_2012Metric_Pad1.20x1.40mm_HandSolder, symbol Device:R
- added R2: 0.003, Resistor_SMD:R_2512_6332Metric, symbol Device:R
- added R5, R6: 51kR, Resistor_SMD:R_0805_2012Metric, symbol Device:R
- added TP1, TP2, TP3, TP4, TP5, TP6, TP7, TP8: ~, TestPoint:TestPoint_Pad_D1.5mm, symbol Connector:TestPoint
- added U1: INA240A1, Package_SO:SOIC-8_3.9x4.9mm_P1.27mm, symbol Amplifier_Current:INA240A3D
- added U4, U8: UCC27211A, Package_SO:TI_SO-PowerPAD-8, symbol Power_Management_IC:UCC27211A
- added U7: STM32F446RETx, Package_QFP:LQFP-64_10x10mm_P0.5mm, symbol MCU_ST_STM32F4:STM32F446RETx
- added Y1: 25MHz, Crystal:Crystal_SMD_3225-4Pin_3.2x2.5mm, symbol Device:Crystal_GND24
- C1: value C -> 5.6n; footprint Capacitor_SMD:C_1210_3225Metric_Pad1.33x2.70mm_HandSolder -> Capacitor_SMD:C_1206_3216Metric; CPN (none) -> GRM3195C2A562JA01D
- D1: value D -> SKL16; footprint Diode_SMD:D_QFN_3.3x3.3mm_P0.65mm -> Diode_SMD:Nexperia_CFP3_SOD-123W; CPN (none) -> SKL16
- L1: renamed from L2; footprint Power_Inductor:VER2923 -> Power_Inductor_THT:VER2923; CPN (none) -> VER2923-223; now left out of the parts list
- R1: value R -> 0.003; footprint Resistor_SMD:R_0805_2012Metric -> Resistor_SMD:R_2512_6332Metric; now left out of the parts list
- U2: renamed from U3; value INA240A3D -> INA240A1; CPN (none) -> INA240A1DR
Connections:
- net GND: now also C10.2, C11.2, C12.2, C13.2, C14.2, C15.2, C16.2, C17.2, C18.2, C19.2, C20.2, C21.2, C22.2, C23.2, C3.2, C31.2, C32.2, C36.2, C38.2, C39.2, C4.1, C40.2, C41.2, C42.2, C43.2, C44.2, C45.2, C46.2, C47.1, C49.1, C5.1, C50.2, C52.2, C53.2, C6.1, C7.1, C8.1, C9.1, D5.1 (A1), D6.1 (A1), H1.1, H2.1, H3.1, H4.1, J1.1 (Pin_1), J2.1 (Pin_1), Q3.1 (S), Q3.2 (S), Q3.3 (S), Q4.1 (S), Q4.2 (S), Q4.3 (S), R11.1, R12.1, R13.1, R16.1, U1.2 (GND), U1.4 (GND), U4.7 (VSS), U4.9 (Pad), U7.12 (VSSA), U7.18 (VSS), U7.31 (VSS), U7.47 (VSS), U7.63 (VSS), U8.7 (VSS), U8.9 (Pad), Y1.2, Y1.4
- net +12V: now reaches R1.2
- net +12V: now also R1.1, C23.1, C3.1, C36.1, C4.2, C5.2, C6.2, C7.2, C8.2, C9.2, D5.2 (A2), D7.2 (A), D8.2 (A), F1.1, F1.2, J1.2 (Pin_2), Q1.5 (D), R5.2, U1.1 (-), U1.8 (+), U4.1 (VDD), U8.1 (VDD); no longer U2.1 (-)
- net +Vref: now reaches U2.3 (REF2)
- net +Vref: now also U2.7 (REF1), C52.1, C53.1, U1.3 (REF2), U1.7 (REF1), U7.21 (PA5)
- net at U2.5: now also R18.2, TP8.1
- net +3.3V: now reaches U2.6 (V+)
- net +3.3V: now also C22.1, C38.1, C39.1, C40.1, C41.1, C42.1, C43.1, C44.1, C45.1, C50.1, FB1.2, U1.6 (V+), U7.19 (VDD), U7.32 (VDD), U7.48 (VDD), U7.64 (VDD)
- net SW1: now reaches L1.1
- net SW1: now also C1.1, C27.2, Q1.1 (S), Q1.2 (S), Q1.3 (S), Q3.5 (D), TP1.1, U4.4 (HS)
- net at D1.2 (A): now also Q1.4 (G), R7.1, TP3.1
- net HO_1: now reaches D1.1 (K)
- net HO_1: now also R7.2, U4.3 (HO); no longer C1.1
- net at C1.2: now also R11.2
- new net: D2.2 (A), Q2.4 (G), R8.1, TP4.1
- new net: R17.1, TP7.1, U1.5
- new net: C2.2, R12.2
- new net: C27.1, D7.1 (K), U4.2 (HB)
- new net: D4.2 (A), Q4.4 (G), R10.1, TP6.1
- new net: C37.1, D8.1 (K), U8.2 (HB)
- new net: D3.2 (A), Q3.4 (G), R9.1, TP5.1
- new net +3.3VA: C19.1, C20.1, C21.1, FB1.1, U7.13 (VDDA)
- new net +36V: C10.1, C11.1, C12.1, C13.1, C14.1, C15.1, C16.1, D6.2 (A2), F2.1, F2.2, J2.2 (Pin_2), Q2.5 (D), R2.1, R2.2, R6.2, U2.1 (-), U2.8 (+)
- new net BOOT: U7.60 (BOOT0)
- new net CAN1_RX: U7.44 (PA11)
- new net CAN1_S: U7.43 (PA10)
- new net CAN1_TX: U7.45 (PA12)
- new net HI_1: U4.5 (HI), U7.41 (PA8)
- new net HI_2: U7.42 (PA9), U8.5 (HI)
- new net HO_2: D2.1 (K), R8.2, U8.3 (HO)
- new net HSEC_IN: C47.2, U7.5 (PH0), Y1.3
- new net HSEC_OUT: C49.2, U7.6 (PH1), Y1.1
- new net I_SENSE_1: C17.1, R17.2, U7.15 (PA1)
- new net I_SENSE_2: C18.1, R18.1, U7.16 (PA2)
- new net LI_1: U4.6 (LI), U7.23 (PA7)
- new net LI_2: U7.26 (PB0), U8.6 (LI)
- new net LO_1: D3.1 (K), R9.2, U4.8 (LO)
- new net LO_2: D4.1 (K), R10.2, U8.8 (LO)
- new net PB1: U7.27 (PB1)
- new net PB10: U7.29 (PB10)
- new net PB2: U7.28 (PB2)
- new net PC0: J4.13 (Pin_13), U7.8 (PC0)
- new net PC1: J4.12 (Pin_12), U7.9 (PC1)
- new net PC10: J4.7 (Pin_7), U7.51 (PC10)
- new net PC11: J4.8 (Pin_8), U7.52 (PC11)
- new net PC12: J4.9 (Pin_9), U7.53 (PC12)
- new net PC13: J4.16 (Pin_16), U7.2 (PC13)
- new net PC14: J4.15 (Pin_15), U7.3 (PC14)
- new net PC15: J4.14 (Pin_14), U7.4 (PC15)
- new net PC2: J4.10 (Pin_10), U7.10 (PC2)
- new net PC3: J4.11 (Pin_11), U7.11 (PC3)
- new net PC4: J4.6 (Pin_6), U7.24 (PC4)
- new net PC5: J4.5 (Pin_5), U7.25 (PC5)
- new net PC6: J4.4 (Pin_4), U7.37 (PC6)
- new net PC7: J4.3 (Pin_3), U7.38 (PC7)
- new net PC8: J4.2 (Pin_2), U7.39 (PC8)
- new net PC9: J4.1 (Pin_1), U7.40 (PC9)
- new net RESET: U7.7 (NRST)
- new net SW2: C2.1, C37.2, L1.2, Q2.1 (S), Q2.2 (S), Q2.3 (S), Q4.5 (D), TP2.1, U8.4 (HS)
- new net SWCLK: U7.49 (PA14)
- new net SWDIO: U7.46 (PA13)
- new net SWO: U7.55 (PB3)
- new net VCAP: C46.1, U7.30 (VCAP_1)
- new net V_1: C32.1, R16.2, R5.1, U7.17 (PA3)
- new net V_2: C31.1, R13.2, R6.1, U7.20 (PA4)
- no-connect marks 0 -> 14
Other:
- added sheet Can_Module (CAN.kicad_sch)
- added sheet Debug (Degug.kicad_sch)
- added sheet Supply (Supply.kicad_sch)
- note added: "fc=160kHz"
- moved on the sheet: L1, U2
